File: Zündung/KiCad/Zuendung/Zuendung.kicad_sch (KiCad schematic)
At the start: 44 parts, among them J1 Conn_01x08_Socket, J1 USB_B_Micro, J3 SWD, Q1 Q_NMOS_DGS, U2 TLV2371DBV, U2 USBLC6-2SC6, U5 TLV2371DBV, U6 TLV2371DBV, U9 STM32G431K8Tx

Commit message: update HW
Parts:
- removed J1: Conn_01x08_Socket, symbol Connector:Conn_01x08_Socket
- added C14: 100n, Capacitor_SMD:C_0603_1608Metric, symbol Device:C
- added C15, C16: 4.7u, Capacitor_SMD:C_0805_2012Metric, symbol Device:C
- added H1, H2: MountingHole_Pad, MountingHole:MountingHole_3.2mm_M3_Pad_Via, symbol Mechanical:MountingHole_Pad
- added J1: Conn_01x04, Connector_Wire:SolderWire-0.75sqmm_1x04_P4.8mm_D1.25mm_OD2.3mm, symbol Connector_Generic:Conn_01x04
- added J5: Conn_01x03, Connector_Wire:SolderWire-0.75sqmm_1x03_P4.8mm_D1.25mm_OD2.3mm, symbol Connector_Generic:Conn_01x03
- added Q2: Q_NMOS_DGS, Package_TO_SOT_SMD:SOT-23-3, symbol Device:Q_NMOS_DGS
- added R18: 22, Resistor_SMD:R_0603_1608Metric, symbol Device:R
- added U7: INA181, Package_TO_SOT_SMD:SOT-23-6, symbol Amplifier_Current:INA181
- C7: value 100n -> 150n; footprint Capacitor_SMD:C_0805_2012Metric -> Capacitor_THT:C_Rect_L32.0mm_W15.0mm_P27.00mm; Hersteller Nr. (none) -> MKP1O131505I00KSSD
- C8: value 100n -> 10n; footprint Capacitor_SMD:C_0805_2012Metric -> Capacitor_THT:C_Rect_L18.0mm_W7.0mm_P15.00mm_FKS3_FKP3; Hersteller Nr. (none) -> MKP1U021004D00MI00
- D2: footprint (none) -> Diode_SMD:D_SOD-123; Hersteller Nr. (none) -> MMSZ5233B-E3-08
- D3: footprint (none) -> Diode_SMD:D_SOD-123; Hersteller Nr. (none) -> MMSZ5242B-E3-08
- D4: footprint (none) -> Package_TO_SOT_THT:TO-220-2_Vertical
- J1: footprint Connector_USB:USB_Mini-B_Lumberg_2486_01_Horizontal -> Connector_USB:USB_Micro-B_Wuerth_614105150721_Vertical; Hersteller Nr. UJ2-MBH-1-SMT-TR -> (none); Info USB Mini B -> (none); Mouser Nr. 490-UJ2-MBH-1-SMT -> (none)
- R2, R3, R4: footprint (none) -> Resistor_SMD:R_0603_1608Metric
- R5: value 0.2 -> 20m; Hersteller Nr. (none) -> ERJ-8CWFR020V
- R6: footprint (none) -> Resistor_THT:R_Axial_DIN0207_L6.3mm_D2.5mm_P10.16mm_Horizontal
- R8: value 10k -> 100; footprint Resistor_SMD:R_0603_1608Metric -> Resistor_SMD:R_1206_3216Metric
Connections:
- net +3V3: now also C14.1, U7.6 (V+)
- net FuelRelay: now also R8.2, J1.3 (Pin_3)
- net GND: now also C14.2, C15.2, C16.2, H1.1, H2.1, J5.3 (Pin_3), Q2.3 (S), U7.2 (GND), U7.4 (-), U7.5 (REF); no longer R8.1
- net Ignition: now also C8.2, J5.1 (Pin_1), J5.2 (Pin_2); no longer C7.2
- net SpeedSignalMinus: now also J1.2 (Pin_2)
- net SpeedSignalPlus: now also J1.1 (Pin_1)
- net Tacho: now also U9.6 (PA1)
- net VCC: now also C15.1, C16.1, J1.4 (Pin_4)
- net at Q1.2 (G), R7.2: no longer R8.2
- net at Q1.3 (S), R5.1: now also U7.3 (+); no longer R12.1
- net at D4.1 (K), R6.2: now also C7.2; no longer C8.2
- net RelayOutput: now reaches U9.11 (PA6)
- net RelayOutput: now also R18.1
- net ISens: now reaches U9.5 (PA0)
- net ISens: now also R12.1, U7.1
- new net: Q2.1 (D), R8.1
- new net: Q2.2 (G), R18.2
- no-connect marks 26 -> 21
Other:
- moved on the sheet: C7, C8, J1, U2

Commit message: update HW
Parts:
- removed D4: D, Package_TO_SOT_THT:TO-220-2_Vertical, symbol Device:D
- removed Q1: Q_NMOS_DGS, symbol Device:Q_NMOS_DGS
- removed Q2: Q_NMOS_DGS, Package_TO_SOT_SMD:SOT-23-3, symbol Device:Q_NMOS_DGS
- removed U2, U5, U6: TLV2371DBV, Package_TO_SOT_SMD:SOT-23-5, symbol Amplifier_Operational:TLV2371DBV
- added C17: 2.2u, Capacitor_SMD:C_0603_1608Metric, symbol Device:C
- added C18: 1u, Capacitor_SMD:C_0603_1608Metric, symbol Device:C
- added C19: 4.7u, Capacitor_SMD:C_0805_2012Metric, symbol Device:C
- added C20: 100n, Capacitor_SMD:C_0805_2012Metric, symbol Device:C
- added D4: 1A/60V, Diode_SMD:D_SMF, symbol Device:D_Schottky
- added H3, H4: MountingHole, MountingHole:MountingHole_3.5mm, symbol Mechanical:MountingHole
- added Q2: DMN6140L, Package_TO_SOT_SMD:SOT-23, symbol Transistor_FET:DMN6140L
- added Q3: Q_NMOS_GDS, Package_TO_SOT_THT:TO-247-3_Vertical, symbol Device:Q_NMOS_GDS
- added U10: TL072, Package_SO:SOIC-8_3.9x4.9mm_P1.27mm, symbol Amplifier_Operational:TL072
- added U2: AP2204RA-3.3, Package_TO_SOT_SMD:SOT-89-3, symbol Regulator_Linear:AP2204RA-3.3
- added unit 3 of U9
- added unit 2 of U9
- C7: footprint Capacitor_THT:C_Rect_L32.0mm_W15.0mm_P27.00mm -> Capacitor_THT:C_Rect_L26.5mm_W6.0mm_P22.50mm_MKS4; Hersteller Nr. MKP1O131505I00KSSD -> MKS4J031505B00MSSD
- C8: footprint Capacitor_THT:C_Rect_L18.0mm_W7.0mm_P15.00mm_FKS3_FKP3 -> Capacitor_THT:C_Rect_L10.0mm_W3.0mm_P7.50mm_MKS4; Hersteller Nr. MKP1U021004D00MI00 -> MKS4J021002B00KSSD
- R6: value 10k -> 3.9; footprint Resistor_THT:R_Axial_DIN0207_L6.3mm_D2.5mm_P10.16mm_Horizontal -> Resistor_THT:R_Axial_DIN0414_L11.9mm_D4.5mm_P15.24mm_Horizontal; Hersteller Nr. (none) -> PR02FS0203908KR500
- R8: value 100 -> 680
- U1: Hersteller Nr. (none) -> RAA2114034GP3#JA0
Connections:
- net +3.3V is gone; now on net +3V3: C2.1, L1.2, U1.1 (Vout)
- net +3V3: now also D4.1 (K)
- net GND: now also C17.2, C18.2, C19.2, C20.2, Q2.2 (S), U10.3 (+), U10.4 (V-), U2.1 (GND), U9.4 (V-), U9.5 (+)
- net Ignition: now also Q3.2 (D)
- net SpeedSignalPlus: now also U10.5 (+)
- net Tacho: now also U9.10 (PA5); no longer U9.6 (PA1)
- net VBUS: now also C18.1, U2.2 (VIN)
- net VCC: now also C19.1, C20.1, U10.8 (V+), U9.8 (V+)
- net at C13.1, R7.1: now also U9.7
- net at R7.2: now also Q3.1 (G)
- net at R13.1, R15.2: now also U9.1
- net at R12.2, R14.1: now also U9.3 (+)
- net at R13.2, R9.1: now also U9.2 (-)
- net at R5.1, U7.3 (+): now also Q3.3 (S)
- net at R15.1, R16.2: now also U9.6 (-)
- net at R3.1: now also U10.6 (-), U10.7
- net at R8.1: now also Q2.3 (D)
- net at R18.2: now also Q2.1 (G)
- new net: C17.1, D4.2 (A), U2.3 (VOUT)
- new net: U10.1, U10.2 (-)
- no-connect marks 21 -> 20
Other:
- moved on the sheet: C1, C13, C14, C2, C5, C6, C7, C8, D1, L1, R1, R12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

Commit message: Hardware finalized
Parts:
- removed C14: 100n, Capacitor_SMD:C_0603_1608Metric, symbol Device:C
- removed U10: TL072, Package_SO:SOIC-8_3.9x4.9mm_P1.27mm, symbol Amplifier_Operational:TL072
- removed U7: INA181, Package_TO_SOT_SMD:SOT-23-6, symbol Amplifier_Current:INA181
- removed unit 3 of U9
- removed unit 2 of U9
- added D5: D_Zener, Diode_SMD:D_SMC, symbol Device:D_Zener
- added Q1: DMN6140L, Package_TO_SOT_SMD:SOT-23, symbol Transistor_FET:DMN6140L
- added U5, U6: OPA990, Package_TO_SOT_SMD:SOT-23-5, symbol Amplifier_Operational:ADA4610-1xRJ
- C13: value 100n -> 100p
- C15, C16: footprint Capacitor_SMD:C_0805_2012Metric -> Capacitor_SMD:C_1206_3216Metric; Hersteller Nr. CL21A475KBQNNNE -> (none)
- C19, C6: Hersteller Nr. (none) -> CL21A475KBQNNNE
- C20, C5: footprint Capacitor_SMD:C_0805_2012Metric -> Capacitor_SMD:C_0603_1608Metric
- Q3: value Q_NMOS_GDS -> MSC090SMA070B
- R12, R13: value 1k -> 100k
- R14: value 1k -> 120
- R15: value 1k -> 0
- R18, R7: value 22 -> 120
Connections:
- net GND: now also R16.2, D5.2 (A), Q1.2 (S), U5.2 (V-), U6.2 (V-); no longer R14.2
- net SpeedSignalPlus: now also U6.3 (+)
- net VCC: now also D5.1 (K), U5.5 (V+), U6.5 (V+)
- net at Q3.1 (G), R7.2: now also R15.2
- net at Q3.3 (S), R5.1: now also R12.1, R13.1
- net at C13.1, R7.1: now also R12.2, U5.1
- net FETOff: now reaches R14.1
- net FETOff: now also U9.8 (PA3); no longer R12.2
- net at R9.1: now also R16.1, U5.3 (+); no longer R13.2
- net at C13.2: now also R13.2, U5.4 (-); no longer R16.1
- net at R3.1: now also U6.1, U6.4 (-)
- net at R15.1: now also Q1.3 (D); no longer R16.2
- net ISens: no longer names the net of U9.5 (PA0)
- net ISens: no longer R12.1
- new net: Q1.1 (G), R14.2
- no-connect marks 20 -> 21
Other:
- moved on the sheet: C19, C20, C5, C6, C7, C8, Q3, R3, R4, R5, R6, R7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
