File: Zuendung/Hardware/Zuendung/Zuendung.kicad_pcb (KiCad board)
At the start: 2 copper layers, 66.5 x 75 mm, 59 parts, among them J1 Conn_01x04, J2 SWD, J3 USB_B_Micro, J5 Conn_01x03, Q1 DMN6140L, Q2 DMN6140L, Q3 MSC090SMA070B, U2 AP2204RA-3.3, U3 USBLC6-2SC6, U4 STM32G431K8Tx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

Commit message: update Hardware
Parts:
- removed H3: MountingHole, MountingHole:MountingHole_3.5mm
- added C14: 10u, Capacitor_SMD:C_0603_1608Metric, F.Cu at (125.5, 119.7)
- added C21: 4.7u, Capacitor_SMD:C_0805_2012Metric, F.Cu at (114.7, 115.3)
- added C22: 100n, Capacitor_SMD:C_0603_1608Metric, F.Cu at (116.5, 115.3)
- added C23: 10n, Capacitor_SMD:C_0603_1608Metric, F.Cu at (128.6, 119.7)
- added C24: 100n, Capacitor_SMD:C_0603_1608Metric, F.Cu at (132.0, 121.2)
- added Q4: BSS83P, Package_TO_SOT_SMD:SOT-23, F.Cu at (114.0, 80.4)
- added R17: 10k, Resistor_SMD:R_0603_1608Metric, F.Cu at (112.8, 76.8)
- added R19: 10k, Resistor_SMD:R_0603_1608Metric, F.Cu at (114.8, 84.0)
- added R20: 10k, Resistor_SMD:R_0603_1608Metric, F.Cu at (113.2, 84.0)
- added R21: 10k, Resistor_SMD:R_0603_1608Metric, F.Cu at (125.5, 118.1)
- added TP1: TachoRaw, TestPoint:TestPoint_Pad_D1.0mm, F.Cu at (118.8, 90.8)
- added TP10: FetOff, TestPoint:TestPoint_Pad_D1.0mm, F.Cu at (140.1, 112.8)
- added TP11: TPDiag2, TestPoint:TestPoint_Pad_D1.0mm, F.Cu at (139.0, 121.8)
- added TP12: ISetDAC, TestPoint:TestPoint_Pad_D1.0mm, F.Cu at (134.8, 118.2)
- added TP2: Tacho, TestPoint:TestPoint_Pad_D1.0mm, F.Cu at (119.6, 110.2)
- added TP3: TachoMean, TestPoint:TestPoint_Pad_D1.0mm, F.Cu at (119.6, 112.4)
- added TP4: 3V3, TestPoint:TestPoint_Pad_D1.0mm, F.Cu at (135.2, 116.0)
- added TP5: FuelRelay, TestPoint:TestPoint_Pad_D1.0mm, F.Cu at (110.6, 79.8)
- added TP6: FuelRelayFet, TestPoint:TestPoint_Pad_D1.0mm, F.Cu at (115.8, 93.1)
- added TP7: ControllerOutput, TestPoint:TestPoint_Pad_D1.0mm, F.Cu at (136.3, 100.1)
- added TP8: ISet, TestPoint:TestPoint_Pad_D1.0mm, F.Cu at (127.5, 102.8)
- added TP9: TPDiag1, TestPoint:TestPoint_Pad_D1.0mm, F.Cu at (136.8, 124.4)
- added U7: OPA990, Package_TO_SOT_SMD:SOT-23-5, F.Cu at (119.5, 115.8)
- moved R4 27.3 mm to (128.6, 118.1), turned to 0 degrees
- moved R3 19.5 mm to (122.0, 112.3)
- moved R8 11.5 mm to (115.0, 76.0), turned to -90 degrees
- moved R18 4.98 mm to (114.0, 90.5)
- moved Q2 4.92 mm to (114.0, 87.7)
- moved H4 4.70 mm to (117.0, 142.0)
- moved R16 1.08 mm to (130.4, 102.3), turned to 90 degrees
- moved H1 0.50 mm to (105.0, 79.5)
- moved H2 0.50 mm to (161.7, 79.5)
- moved C19 0.45 mm to (133.6, 98.4)
- moved C20 0.45 mm to (133.8, 100.2)
Connections:
- R8 pad 1: Net-(Q2-D) -> FuelRelay
- R8 pad 2: FuelRelay -> Net-(Q4-D)
- U4 pad 12: unconnected-(U4-PA7-Pad12) -> Net-(U4-PA7)
- U4 pad 6: unconnected-(U4-PA1-Pad6) -> Net-(U4-PA1)
- U4 pad 7: unconnected-(U4-PA2-Pad7) -> Net-(U4-PA2)
Routing:
- net VCC: track 89.2 -> 116.7 mm, vias 3 -> 5
- net Net-(U6--): track 8.95 -> 29.6 mm
- net GND: track 140.0 -> 121.5 mm, vias 100 -> 111
- net RelayOutput: track 33.5 -> 48.1 mm, vias 0 -> 2
- net Tacho: track 34.5 -> 21.0 mm
- net Tacho_MeanValue: track 0.00 -> 11.4 mm
- net Net-(U4-PA2): track 0.00 -> 11.1 mm
- net Net-(U4-PA1): track 0.00 -> 8.12 mm
- net Net-(Q4-D): track 0.00 -> 5.10 mm
- net Net-(U4-PA7): track 0.00 -> 4.76 mm
- net Net-(Q4-G): track 0.00 -> 4.68 mm
- net Net-(U5-+): track 4.61 -> 7.68 mm
- net +3V3: track 90.1 -> 92.2 mm
- net Net-(C13-Pad1): track 7.44 -> 9.41 mm
- net FETOff: track 20.5 -> 21.8 mm
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Other:
- board size 66.5 x 75 mm -> 66.5 x 81 mm

Commit message: Update Hardware
Parts:
- removed C21: 4.7u, Capacitor_SMD:C_0805_2012Metric
- removed C22: 100n, Capacitor_SMD:C_0603_1608Metric
- removed U7: OPA990, Package_TO_SOT_SMD:SOT-23-5
- added R22: 6.8k, Resistor_SMD:R_0603_1608Metric, F.Cu at (124.8, 116.9)
- added R23: 1.8k, Resistor_SMD:R_0603_1608Metric, F.Cu at (125.5, 119.2)
- R21: value 10k -> 6.8k
- R3: value 40k -> 6.8k
- R4: value 10k -> 1.8k
- moved R3 9.55 mm to (128.6, 119.2), turned to 180 degrees
- moved TP3 6.83 mm to (120.2, 119.2)
- moved TP2 6.72 mm to (120.1, 116.9)
- moved C10 2.70 mm to (129.7, 133.4)
- moved J2 2.70 mm to (112.7, 133.3)
- moved R11 2.70 mm to (127.5, 135.4)
- moved C11 2.70 mm to (120.1, 123.9)
- moved C14 2.70 mm to (125.5, 122.4)
- moved C18 2.70 mm to (108.8, 125.5)
- moved C23 2.70 mm to (128.6, 122.4)
- moved C24 2.70 mm to (132.0, 123.9)
- moved D4 2.70 mm to (112.2, 121.8)
- moved R21 2.70 mm to (125.5, 120.8)
- moved R4 2.70 mm to (128.6, 120.8)
- moved TP11 2.70 mm to (139.0, 124.5)
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Routing:
- net VCC: track 116.7 -> 95.4 mm, vias 5 -> 3
- net Net-(U6--): track 29.6 -> 43.7 mm
- net Tacho: track 21.0 -> 16.0 mm
- net Tacho_MeanValue: track 11.4 -> 7.60 mm
- net GND: track 121.5 -> 124.8 mm, vias 111 -> 106
- net FETOff: track 21.8 -> 24.5 mm
- net USet: track 26.3 -> 29.0 mm
- net RelayOutput: track 48.1 -> 50.8 mm
- net +3V3: track 92.2 -> 94.7 mm

Commit message: udpdate Hardware
Parts:
- removed C24: 100n, Capacitor_SMD:C_0603_1608Metric
- R16: value 1k -> 1
- R7: value 120 -> 750
- R9: value 1k -> 2.4k
- TP3: value TachoMean -> TachoMV
Changed lines of the file:
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@@
     (property "ki_keywords" "cap capacitor")
     (attr smd)
-    (fp_text reference "C23" (at -3.15 0.7) (layer "F.SilkS")
+    (fp_text reference "C23" (at -3 0) (layer "F.SilkS")
         (effects (font (size 1 1) (thickness 0.15)))
     )
@@
     (property "ki_keywords" "R res resistor")
     (attr smd)
-    (fp_text reference "R4" (at 2.8 -0.3) (layer "F.SilkS")
+    (fp_text reference "R4" (at 2.6 0) (layer "F.SilkS")
         (effects (font (size 1 1) (thickness 0.15)))
     )
@@
     )
   )
-  (footprint "Capacitor_SMD:C_0603_1608Metric" (layer "F.Cu")
-    (at 132 123.925 -90)
-    (descr "Capacitor SMD 0603 (1608 Metric), square (rectangular) end terminal, IPC_7351 nominal, (Body size source: IPC-SM-782 page 76, https://www.pcb-3d.com/wordpress/wp-content/uploads/ipc-sm-782a_amendment_1_and_2.pdf), generated with kicad-footprint-generator")
-    (tags "capacitor")
-    (property "Hersteller Nr." "885382206004")
-    (property "Info" "0.1uF; 50V, X7R; -55C;+125C")
-    (property "Mouser Nr." "710-885382206004")
-    (property "Sheetfile" "Zuendung.kicad_sch")
-    (property "Sheetname" "")
-    (property "ki_description" "Unpolarized capacitor")
-    (property "ki_keywords" "cap capacitor")
-    (attr smd)
-    (fp_text reference "C24" (at 0 -1.75 90) (layer "F.SilkS")
-        (effects (font (size 1 1) (thickness 0.15)))
-    )
-    (fp_text value "100n" (at 0 1.43 90) (layer "F.Fab")
-        (effects (font (size 1 1) (thickness 0.15)))
-    )
-    (fp_text user "${REFERENCE}" (at 0 0 90) (layer "F.Fab")
-        (effects (font (size 0.4 0.4) (thickness 0.06)))
-    )
-    (fp_line (start -0.14058 -0.51) (end 0.14058 -0.51)
-      (stroke (width 0.12) (type solid)) (layer "F.SilkS"))
-    (fp_line (start -0.14058 0.51) (end 0.14058 0.51)
-      (stroke (width 0.12) (type solid)) (layer "F.SilkS"))
-    (fp_line (start -1.48 -0.73) (end 1.48 -0.73)
-      (stroke (width 0.05) (type solid)) (layer "F.CrtYd"))
-    (fp_line (start -1.48 0.73) (end -1.48 -0.73)
-      (stroke (width 0.05) (type solid)) (layer "F.CrtYd"))
-    (fp_line (start 1.48 -0.73) (end 1.48 0.73)
-      (stroke (width 0.05) (type solid)) (layer "F.CrtYd"))
-    (fp_line (start 1.48 0.73) (end -1.48 0.73)
-      (stroke (width 0.05) (type solid)) (layer "F.CrtYd"))
-    (fp_line (start -0.8 -0.4) (end 0.8 -0.4)
-      (stroke (width 0.1) (type solid)) (layer "F.Fab"))
-    (fp_line (start -0.8 0.4) (end -0.8 -0.4)
-      (stroke (width 0.1) (type solid)) (layer "F.Fab"))
-    (fp_line (start 0.8 -0.4) (end 0.8 0.4)
-      (stroke (width 0.1) (type solid)) (layer "F.Fab"))
-    (fp_line (start 0.8 0.4) (end -0.8 0.4)
-      (stroke (width 0.1) (type solid)) (layer "F.Fab"))
-    (pad "1" smd roundrect (at -0.775 0 270) (size 0.9 0.95) (layers "F.Cu" "F.Paste" "F.Mask") (roundrect_rratio 0.25)
-      (net 2 "GND") (pintype "passive"))
-    (pad "2" smd roundrect (at 0.775 0 270) (size 0.9 0.95) (layers "F.Cu" "F.Paste" "F.Mask") (roundrect_rratio 0.25)
-      (net 18 "USet") (pintype "passive"))
-    (model "${KICAD6_3DMODEL_DIR}/Capacitor_SMD.3dshapes/C_0603_1608Metric.wrl"
-      (offset (xyz 0 0 0))
-      (scale (xyz 1 1 1))
-      (rotate (xyz 0 0 0))
-    )
-  )
   (footprint "Resistor_SMD:R_0603_1608Metric" (layer "F.Cu")
     (at 130.4 102.3 90)
@@
         (effects (font (size 1 1) (thickness 0.15)))
     )
-    (fp_text value "1k" (at 0 1.43 90) (layer "F.Fab")
+    (fp_text value "1" (at 0 1.43 90) (layer "F.Fab")
         (effects (font (size 1 1) (thickness 0.15)))
     )
@@
         (effects (font (size 1 1) (thickness 0.15)))
     )
-    (fp_text value "TachoMean" (at 0 1.55) (layer "F.Fab")
+    (fp_text value "TachoMV" (at 0 1.55) (layer "F.Fab")
         (effects (font (size 1 1) (thickness 0.15)))
     )
@@
     (property "ki_keywords" "R res resistor")
     (attr smd)
-    (fp_text reference "R3" (at -2.8 0.1) (layer "F.SilkS")
+    (fp_text reference "R3" (at -2.6 0) (layer "F.SilkS")
         (effects (font (size 1 1) (thickness 0.15)))
     )
@@
         (effects (font (size 1 1) (thickness 0.15)))
     )
-    (fp_text value "120" (at 0 1.43) (layer "F.Fab")
+    (fp_text value "750" (at 0 1.43) (layer "F.Fab")
         (effects (font (size 1 1) (thickness 0.15)))
     )
@@
         (effects (font (size 1 1) (thickness 0.15)))
     )
-    (fp_text value "1k" (at 0 1.43) (layer "F.Fab")
-        (effects (font (size 1 1) (thickness 0.15)))
-    )
+    (fp_text value "2.4k" (at 0 1.43) (layer "F.Fab")
+        (effects (font (size 1 1) (thickness 0.15)))
+    )
