File: Zuendung/Hardware/Zuendung/Zuendung.kicad_sch (KiCad schematic)
At the start: 59 parts, among them J1 Conn_01x04, J1 USB_B_Micro, J3 SWD, J5 Conn_01x03, Q1 DMN6140L, Q2 DMN6140L, Q3 MSC090SMA070B, U2 AP2204RA-3.3, U2 USBLC6-2SC6, U5 OPA990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

Commit message: changes for Version 2.0
Parts:
- added C1: 10u, Capacitor_SMD:C_0603_1608Metric, symbol Device:C
- added C21: 4.7u, Capacitor_SMD:C_0805_2012Metric, symbol Device:C
- added C22: 100n, Capacitor_SMD:C_0603_1608Metric, symbol Device:C
- added Q4: BSS83P, Package_TO_SOT_SMD:SOT-23, symbol Transistor_FET:BSS83P
- added R17, R19, R20, R21: 10k, Resistor_SMD:R_0603_1608Metric, symbol Device:R
- added U7: OPA990, Package_TO_SOT_SMD:SOT-23-5, symbol Amplifier_Operational:ADA4610-1xRJ
Connections:
- net FuelRelay: now also R8.1; no longer R8.2
- net GND: now also C1.1, C21.2, C22.2, R17.2, U7.2 (V-)
- net Tacho: now also U7.3 (+)
- net VCC: now also C21.1, C22.1, Q4.2 (S), R19.1, U7.5 (V+)
- net at Q2.3 (D): now also R20.2; no longer R8.1
- net at U9.3 (PF1): now also C1.2, R21.2
- new net: Q4.1 (G), R19.2, R20.1
- new net: Q4.3 (D), R17.1, R8.2
- new net Tacho_MeanValue: R21.1, U7.1, U7.4 (-)
- no-connect marks 21 -> 20
Other:
- moved on the sheet: C1, C13, C19, C20, C3, C4, C5, C6, C7, C8, D2, D3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

Commit message: update Hardware
Parts:
- removed H3: MountingHole, MountingHole:MountingHole_3.5mm, symbol Mechanical:MountingHole
- added C1: 100n, Capacitor_SMD:C_0603_1608Metric, symbol Device:C
- added C23: 10n, Capacitor_SMD:C_0603_1608Metric, symbol Device:C
- added TP1: TachoRaw, TestPoint:TestPoint_Pad_D1.0mm, symbol Connector:TestPoint
- added TP10: FetOff, TestPoint:TestPoint_Pad_D1.0mm, symbol Connector:TestPoint
- added TP11: TPDiag2, TestPoint:TestPoint_Pad_D1.0mm, symbol Connector:TestPoint
- added TP12: ISetDAC, TestPoint:TestPoint_Pad_D1.0mm, symbol Connector:TestPoint
- added TP2: Tacho, TestPoint:TestPoint_Pad_D1.0mm, symbol Connector:TestPoint
- added TP3: TachoMean, TestPoint:TestPoint_Pad_D1.0mm, symbol Connector:TestPoint
- added TP4: 3V3, TestPoint:TestPoint_Pad_D1.0mm, symbol Connector:TestPoint
- added TP5: FuelRelay, TestPoint:TestPoint_Pad_D1.0mm, symbol Connector:TestPoint
- added TP6: FuelRelayFet, TestPoint:TestPoint_Pad_D1.0mm, symbol Connector:TestPoint
- added TP7: ControllerOutput, TestPoint:TestPoint_Pad_D1.0mm, symbol Connector:TestPoint
- added TP8: ISet, TestPoint:TestPoint_Pad_D1.0mm, symbol Connector:TestPoint
- added TP9: TPDiag1, TestPoint:TestPoint_Pad_D1.0mm, symbol Connector:TestPoint
Connections:
- net +3V3: now also TP4.1
- net FETOff: now also TP10.1
- net FuelRelay: now also TP5.1
- net GND: now also C1.1, C23.1
- net RelayOutput: now also TP6.1
- net Tacho: now also C23.2, TP2.1
- net Tacho_MeanValue: now also TP3.1
- net USet: now also C1.2, TP12.1
- net at C13.1, R12.2, R7.1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: now also TP7.1
- net at R3.1, U6.1, U6.4 (-): now also TP1.1
- net at R16.1, R9.1, U5.3 (+): now also TP8.1
- net at C1.2, R21.2: now also U9.12 (PA7); no longer U9.3 (PF1)
- net at U9.6 (PA1): now also TP9.1
- net at U9.7 (PA2): now also TP11.1
- no-connect marks 20 -> 14
Other:
- moved on the sheet: C1, C21, C22, J3, R21, R3, R4, U7, U9

Commit message: Update Hardware
Parts:
- removed C21: 4.7u, Capacitor_SMD:C_0805_2012Metric, symbol Device:C
- removed C22: 100n, Capacitor_SMD:C_0603_1608Metric, symbol Device:C
- removed U7: OPA990, Package_TO_SOT_SMD:SOT-23-5, symbol Amplifier_Operational:ADA4610-1xRJ
- added R22: 6.8k, Resistor_SMD:R_0603_1608Metric, symbol Device:R
- added R23: 1.8k, Resistor_SMD:R_0603_1608Metric, symbol Device:R
- R21: value 10k -> 6.8k
- R3: value 40k -> 6.8k
- R4: value 10k -> 1.8k
- TP3: value TachoMean -> TachoMV
Connections:
- net GND: now also R23.2
- net Tacho_MeanValue: now also R22.2, R23.1
- net at R3.1, TP1.1, U6.1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: now also R22.1
Other:
- moved on the sheet: C23, R3, R4, TP10, TP2, TP3

Commit message: udpdate Hardware
Parts:
- removed C1: 100n, Capacitor_SMD:C_0603_1608Metric, symbol Device:C
- R16: value 1k -> 100
- R7: value 120 -> 750
- R9: value 1k -> 2.4k
Changed lines of the file:
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@@
-    (stroke (width 0) (type default))
-  )
-  (wire (pts (xy 170.18 41.91) (xy 170.18 44.45))
     (stroke (width 0) (type default))
   )
@@
   )
   (wire (pts (xy 219.71 44.45) (xy 219.71 46.99))
-    (stroke (width 0) (type default))
-  )
-  (wire (pts (xy 170.18 52.07) (xy 170.18 55.88))
     (stroke (width 0) (type default))
   )
@@
       (effects (font (size 1.27 1.27)))
     )
-    (property "Value" "120" (at 229.87 41.91 90)
+    (property "Value" "750" (at 229.87 41.91 90)
       (effects (font (size 1.27 1.27)))
     )
@@
     )
   )
-  (symbol (lib_id "Device:C") (at 170.18 48.26 180) (unit 1)
+  (symbol (lib_id "power:+3V3") (at 218.44 97.79 0) (unit 1)
+    (in_bom yes) (on_board yes) (dnp no) (fields_autoplaced)
+    (property "Reference" "#PWR011" (at 218.44 101.6 0)
+      (effects (font (size 1.27 1.27)) hide)
+    )
+    (property "Value" "+3V3" (at 218.44 94.2881 0)
+      (effects (font (size 1.27 1.27)))
+    )
+    (property "Footprint" "" (at 218.44 97.79 0)
+      (effects (font (size 1.27 1.27)) hide)
+    )
+    (property "Datasheet" "" (at 218.44 97.79 0)
+      (effects (font (size 1.27 1.27)) hide)
+    )
+    (pin "1")
+    (instances
+      (project "BallBalancer"
+        (path "/d139795d-9e27-4394-be32-ac05c337c17d/97f62c80-ac17-4829-9f2c-b4ea071a8da4"
+          (reference "#PWR011") (unit 1)
+        )
+      )
+      (project "Zuendung"
+        (path "/f66e51c4-2d7c-4397-97df-35b6b0b0d40b"
+          (reference "#PWR024") (unit 1)
+        )
+      )
+    )
+  )
+  (symbol (lib_id "Amplifier_Operational:ADA4610-1xRJ") (at 195.58 44.45 0) (unit 1)
     (in_bom yes) (on_board yes) (dnp no)
-    (property "Reference" "C1" (at 163.7792 48.26 90)
-      (effects (font (size 1.27 1.27)))
-    )
-    (property "Value" "100n" (at 166.0906 48.26 90)
-      (effects (font (size 1.27 1.27)))
-    )
-    (property "Footprint" "Capacitor_SMD:C_0603_1608Metric" (at 169.2148 44.45 0)
-      (effects (font (size 1.27 1.27)) hide)
-    )
-    (property "Datasheet" "https://www.mouser.ch/datasheet/2/585/MLCC-1837944.pdf" (at 170.18 48.26 0)
-      (effects (font (size 1.27 1.27)) hide)
-    )
-    (property "Hersteller Nr." "885382206004" (at 170.18 48.26 0)
-      (effects (font (size 1.27 1.27)) hide)
-    )
-    (property "Mouser Nr." "710-885382206004" (at 170.18 48.26 0)
-      (effects (font (size 1.27 1.27)) hide)
-    )
-    (property "Info" "0.1uF; 50V, X7R; -55C;+125C" (at 170.18 48.26 0)
+    (property "Reference" "U5" (at 196.85 35.56 0)
+      (effects (font (size 1.27 1.27)))
+    )
+    (property "Value" "OPA990" (at 199.39 38.1 0)
+      (effects (font (size 1.27 1.27)))
+    )
+    (property "Footprint" "Package_TO_SOT_SMD:SOT-23-5" (at 193.04 49.53 0)
+      (effects (font (size 1.27 1.27)) (justify left) hide)
+    )
+    (property "Datasheet" "" (at 195.58 39.37 0)
+      (effects (font (size 1.27 1.27)) hide)
+    )
+    (pin "2")
+    (pin "5")
+    (pin "1")
+    (pin "3")
+    (pin "4")
+    (instances
+      (project "Zuendung"
+        (path "/f66e51c4-2d7c-4397-97df-35b6b0b0d40b"
+          (reference "U5") (unit 1)
+        )
+      )
+    )
+  )
+  (symbol (lib_id "Device:C") (at 200.66 110.49 180) (unit 1)
+    (in_bom yes) (on_board yes) (dnp no)
+    (property "Reference" "C1" (at 194.2592 110.49 90)
+      (effects (font (size 1.27 1.27)))
+    )
+    (property "Value" "100n" (at 196.5706 110.49 90)
+      (effects (font (size 1.27 1.27)))
+    )
+    (property "Footprint" "Capacitor_SMD:C_0603_1608Metric" (at 199.6948 106.68 0)
+      (effects (font (size 1.27 1.27)) hide)
+    )
+    (property "Datasheet" "https://www.mouser.ch/datasheet/2/585/MLCC-1837944.pdf" (at 200.66 110.49 0)
+      (effects (font (size 1.27 1.27)) hide)
+    )
+    (property "Hersteller Nr." "885382206004" (at 200.66 110.49 0)
+      (effects (font (size 1.27 1.27)) hide)
+    )
+    (property "Mouser Nr." "710-885382206004" (at 200.66 110.49 0)
+      (effects (font (size 1.27 1.27)) hide)
+    )
+    (property "Info" "0.1uF; 50V, X7R; -55C;+125C" (at 200.66 110.49 0)
       (effects (font (size 1.27 1.27)) hide)
     )
@@
       (project "Zuendung"
         (path "/f66e51c4-2d7c-4397-97df-35b6b0b0d40b"
-          (reference "C24") (unit 1)
-        )
-      )
-    )
-  )
-  (symbol (lib_id "power:+3V3") (at 218.44 97.79 0) (unit 1)
-    (in_bom yes) (on_board yes) (dnp no) (fields_autoplaced)
-    (property "Reference" "#PWR011" (at 218.44 101.6 0)
-      (effects (font (size 1.27 1.27)) hide)
-    )
-    (property "Value" "+3V3" (at 218.44 94.2881 0)
-      (effects (font (size 1.27 1.27)))
-    )
-    (property "Footprint" "" (at 218.44 97.79 0)
-      (effects (font (size 1.27 1.27)) hide)
-    )
-    (property "Datasheet" "" (at 218.44 97.79 0)
-      (effects (font (size 1.27 1.27)) hide)
-    )
-    (pin "1")
-    (instances
-      (project "BallBalancer"
-        (path "/d139795d-9e27-4394-be32-ac05c337c17d/97f62c80-ac17-4829-9f2c-b4ea071a8da4"
-          (reference "#PWR011") (unit 1)
-        )
-      )
-      (project "Zuendung"
-        (path "/f66e51c4-2d7c-4397-97df-35b6b0b0d40b"
-          (reference "#PWR024") (unit 1)
-        )
-      )
-    )
-  )
-  (symbol (lib_id "Amplifier_Operational:ADA4610-1xRJ") (at 195.58 44.45 0) (unit 1)
-    (in_bom yes) (on_board yes) (dnp no)
-    (property "Reference" "U5" (at 196.85 35.56 0)
-      (effects (font (size 1.27 1.27)))
-    )
-    (property "Value" "OPA990" (at 199.39 38.1 0)
-      (effects (font (size 1.27 1.27)))
-    )
-    (property "Footprint" "Package_TO_SOT_SMD:SOT-23-5" (at 193.04 49.53 0)
-      (effects (font (size 1.27 1.27)) (justify left) hide)
-    )
-    (property "Datasheet" "" (at 195.58 39.37 0)
-      (effects (font (size 1.27 1.27)) hide)
-    )
-    (pin "2")
-    (pin "5")
-    (pin "1")
-    (pin "3")
-    (pin "4")
-    (instances
-      (project "Zuendung"
-        (path "/f66e51c4-2d7c-4397-97df-35b6b0b0d40b"
-          (reference "U5") (unit 1)
-        )
-      )
-    )
-  )
-  (symbol (lib_id "Device:C") (at 200.66 110.49 180) (unit 1)
-    (in_bom yes) (on_board yes) (dnp no)
-    (property "Reference" "C1" (at 194.2592 110.49 90)
-      (effects (font (size 1.27 1.27)))
-    )
-    (property "Value" "100n" (at 196.5706 110.49 90)
-      (effects (font (size 1.27 1.27)))
-    )
-    (property "Footprint" "Capacitor_SMD:C_0603_1608Metric" (at 199.6948 106.68 0)
-      (effects (font (size 1.27 1.27)) hide)
-    )
-    (property "Datasheet" "https://www.mouser.ch/datasheet/2/585/MLCC-1837944.pdf" (at 200.66 110.49 0)
-      (effects (font (size 1.27 1.27)) hide)
-    )
-    (property "Hersteller Nr." "885382206004" (at 200.66 110.49 0)
-      (effects (font (size 1.27 1.27)) hide)
-    )
-    (property "Mouser Nr." "710-885382206004" (at 200.66 110.49 0)
-      (effects (font (size 1.27 1.27)) hide)
-    )
-    (property "Info" "0.1uF; 50V, X7R; -55C;+125C" (at 200.66 110.49 0)
-      (effects (font (size 1.27 1.27)) hide)
-    )
-    (pin "1")
-    (pin "2")
-    (instances
-      (project "BallBalancer"
-        (path "/d139795d-9e27-4394-be32-ac05c337c17d/97f62c80-ac17-4829-9f2c-b4ea071a8da4"
-          (reference "C1") (unit 1)
-        )
-      )
-      (project "Spanner"
-        (path "/ed8d0ee4-83e3-4807-8850-ea20e8975bf5/cb73e00e-b752-4474-a136-20146bf8e401"
-          (reference "C4") (unit 1)
-        )
-      )
-      (project "Zuendung"
-        (path "/f66e51c4-2d7c-4397-97df-35b6b0b0d40b"
           (reference "C9") (unit 1)
         )
@@
       (effects (font (size 1.27 1.27)) (justify left))
     )
-    (property "Value" "1k" (at 182.88 51.435 0)
+    (property "Value" "100" (at 182.88 51.435 0)
       (effects (font (size 1.27 1.27)) (justify left))
     )
@@
       (effects (font (size 1.27 1.27)))
     )
-    (property "Value" "1k" (at 175.26 39.37 90)
+    (property "Value" "2.4k" (at 175.26 39.37 90)
       (effects (font (size 1.27 1.27)))
     )
@@
         )
       )
-    )
-  )
-  (symbol (lib_id "power:GND") (at 170.18 55.88 0) (unit 1)
-    (in_bom yes) (on_board yes) (dnp no) (fields_autoplaced)
-    (property "Reference" "#PWR051" (at 170.18 62.23 0)
-      (effects (font (size 1.27 1.27)) hide)
-    )
-    (property "Value" "GND" (at 170.18 60.96 0)
-      (effects (font (size 1.27 1.27)))
-    )
-    (property "Footprint" "" (at 170.18 55.88 0)
-      (effects (font (size 1.27 1.27)) hide)
-    )
-    (property "Datasheet" "" (at 170.18 55.88 0)
-      (effects (font (size 1.27 1.27)) hide)
-    )
-    (pin "1")
-    (instances
-      (project "Zuendung"
-        (path "/f66e51c4-2d7c-4397-97df-35b6b0b0d40b"
-          (reference "#PWR051") (unit 1)
-        )
-      )
